File: PCB/corneec/OG_mounting_plate.kicad_pcb (KiCad board)
At the start: 2 copper layers, 132.9 x 91.4 mm, 27 parts, among them SW2 KEY_SWITCH

Commit message: Update of rev commit to include extra screw mount
Parts:
- added ?: , kbd:M2_Hole_TH, F.Cu at (143.7, 65.7)
Changed lines of the file:
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@@
     (fp_line (start 9.525 -9.525) (end -9.525 -9.525) (layer "F.Fab") (width 0.15))
+  )
+  (footprint "kbd:M2_Hole_TH" (layer "F.Cu")
+    (at 143.675 65.65)
+    (attr through_hole)
+    (fp_text reference "" (at 0 -3.2) (layer "F.SilkS")
+      (effects (font (size 1 1) (thickness 0.15)))
+    )
+    (fp_text value "" (at 0 3.2) (layer "F.Fab")
+      (effects (font (size 1 1) (thickness 0.15)))
+    )
+    (fp_text user "${REFERENCE}" (at 0.3 0) (layer "F.Fab")
+      (effects (font (size 1 1) (thickness 0.15)))
+    )
+    (pad "" thru_hole circle locked (at 0 0) (size 4.2 4.2) (drill 2.3) (layers *.Cu *.Mask)
+      (net 1 "GNDA"))
   )
   (footprint "kbd:SW_Hole" (layer "F.Cu")
