File: PCB/corneec/corneec.kicad_sch (KiCad schematic)
At the start: 45 parts, among them J1 OLED, J2 MJ-4PP-9, Q1 Q_NMOS_GSD, SW1 SW_Push, SW10 EC_SW, SW11 EC_SW, SW12 EC_SW, SW13 EC_SW, SW14 EC_SW, SW15 EC_SW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

Commit message: Update
Other:
- note added: "Analog Sensing circuit"
- note added: "BLE Status LED"
- note added: "EC Switch Matrix"
- note added: "NOTE: - in order to controll the output of the sensing circuit you can change the value of R10 to fit a higer/lower gain of the OpAmp. - Q1 and R8 can be obmitted"
- note added: "Populate only if using BLE Pro Micro"
- note added: "Power flags"
- note added: "Pro Micro"
- note added: "TRRS"
- title: (none) -> Corne EC Revival
- moved on the sheet: C1, C2, C3, D1, J1, J2, JP1, Q1, R1, R10, R11, R2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

Commit message: Add of standard mounting compatible PCBs
Other:
- note added: "NOTE alternative OpAmp parts might be the following: - TLV9001S"
Changed lines of the file:
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@@
+    (stroke (width 0) (type default) (color 0 0 0 0))
+  )
+  (polyline (pts (xy 138.43 111.76) (xy 138.43 121.92))
     (stroke (width 0) (type default) (color 0 0 0 0))
   )
@@
     (stroke (width 0) (type default) (color 0 0 0 0))
   )
+  (polyline (pts (xy 187.96 121.92) (xy 187.96 111.76))
+    (stroke (width 0) (type default) (color 0 0 0 0))
+  )
   (wire (pts (xy 162.56 134.62) (xy 162.56 130.81))
     (stroke (width 0) (type default) (color 0 0 0 0))
@@
   )
   (wire (pts (xy 184.15 67.31) (xy 184.15 69.85))
+    (stroke (width 0) (type default) (color 0 0 0 0))
+  )
+  (polyline (pts (xy 138.43 111.76) (xy 187.96 111.76))
     (stroke (width 0) (type default) (color 0 0 0 0))
   )
@@
     (effects (font (size 1.27 1.27)) (justify left bottom))
   )
+  (text "NOTE\nalternative OpAmp parts might be the following:\n- TLV9001S"
+    (at 139.7 119.38 0)
+    (effects (font (size 1.27 1.27)) (justify left bottom))
+  )

Commit message: PCB Update and STEP upload
Parts:
- R10: value 22k -> 22k : 100k
Changed lines of the file:
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@@
     (in_bom yes) (on_board yes)
     (property "Reference" "R10" (id 0) (at 167.64 148.4122 90))
-    (property "Value" "22k" (id 1) (at 167.64 150.7236 90))
+    (property "Value" "22k : 100k" (id 1) (at 167.64 150.7236 90))
     (property "Footprint" "cipulot_parts:R_0603_1608Metric_Pad0.98x0.95mm_HandSolder" (id 2) (at 167.64 155.448 90)
       (effects (font (size 1.27 1.27)) hide)
@@
     )
     (path "/00000000-0000-0000-0000-000061d28452"
-      (reference "R10") (unit 1) (value "22k") (footprint "cipulot_parts:R_0603_1608Metric_Pad0.98x0.95mm_HandSolder")
+      (reference "R10") (unit 1) (value "22k : 100k") (footprint "cipulot_parts:R_0603_1608Metric_Pad0.98x0.95mm_HandSolder")
     )
     (path "/add742ad-d41a-4d30-bf31-04e5bebdc9d3"
