File: PCB/OG_mounting_left.kicad_pcb (KiCad board)
At the start: 2 copper layers, 133.8 x 91.4 mm, 54 parts, among them J1 OLED, J2 MJ-4PP-9, Q1 Q_NMOS_GSD, SW1 SW_Push, SW10 EC_SW, SW11 EC_SW, SW12 EC_SW, SW13 EC_SW, SW14 EC_SW, SW15 EC_SW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

Commit message: Update files for JLC production (minimal assembly)
Other:
- board text added: "*"
