File: hardware/pcb/keyboard/keyboard_right.kicad_pcb (KiCad board)
At the start: 2 copper layers, 133.8 x 110.4 mm, 117 parts, among them J1 SM04B-SRSS-TB, J2 PJ320D, J3 HRO_TYPE-C-31-M-12, J4 FH34SRJ-10S-0.5SH, Q1 AO3407, SW1 EC_SW, SW10 EC_SW, SW11 EC_SW, SW12 EC_SW, SW13 EC_SW, SW14 EC_SW, SW15 EC_SW, SW16 EC_SW, SW17 EC_SW, SW18 EC_SW, SW19 EC_SW, SW2 EC_SW, SW20 EC_SW, SW21 EC_SW, SW22 EC_SW, SW23 EC_SW, SW24 EC_SW, SW25 EC_SW, SW26 EC_SW, SW27 EC_SW, SW28 EC_SW, SW29 SW_Push, SW3 EC_SW, SW4 EC_SW, SW5 EC_SW, SW6 EC_SW, SW7 EC_SW, SW8 EC_SW, SW9 EC_SW, U1 74HC4051, U2 OPA350UA, U3 nRF52840_holyiot_18010, U4 XC6220B331MR-G, U5 DT1446-04S, U6 DT1446-04S, U8 TP4054

Commit message: Init STM32G0 PCB
Parts:
- removed D2: LED 0603 RED, LED_SMD:LED_0603_1608Metric
- removed D3: 1N5819, PCM_Diode_SMD_AKL:D_SOD-123
- removed the H16 at (89.1, 75.0)
- removed H19: ~, ec_parts:SMT-SO-M1.6-screwhole_only
- removed J5: ~, ec_parts:PinHeader_1x04_P2.54mm_top_only
- removed J6: ~, ec_parts:PinHeader_1x02_P2.00mm_Vertical
- removed JP1: ~, ec_parts:P1.3mm_Bridged_RoundedPad1.0x1.5mm
- removed Q1: AO3407, PCM_Package_TO_SOT_SMD_AKL:SOT-23
- removed R1: 10k, PCM_Resistor_SMD_AKL:R_0603_1608Metric_Pad0.98x0.95mm
- removed R11: 820K, PCM_Resistor_SMD_AKL:R_0603_1608Metric_Pad0.98x0.95mm
- removed R12: 2M, PCM_Resistor_SMD_AKL:R_0603_1608Metric_Pad0.98x0.95mm
- removed R13: 1k, PCM_Resistor_SMD_AKL:R_0603_1608Metric_Pad0.98x0.95mm
- removed R15: RPROG, PCM_Resistor_SMD_AKL:R_0603_1608Metric_Pad0.98x0.95mm
- removed the R3 at (83.4, 70.1)
- removed U6: DT1446-04S, PCM_Package_TO_SOT_SMD_AKL:SOT-363_SC-70-6_Handsoldering
- removed U8: TP4054, PCM_Package_TO_SOT_SMD_AKL:SOT-23-5
- added C1: 0.1uF, PCM_Capacitor_SMD_AKL:C_0603_1608Metric_Pad1.05x0.95mm, F.Cu at (87.0, 31.9)
- added C6: 5.6p, PCM_Capacitor_SMD_AKL:C_0603_1608Metric_Pad1.05x0.95mm, F.Cu at (75.1, 72.8)
- added C7: 5.6p, PCM_Capacitor_SMD_AKL:C_0603_1608Metric_Pad1.05x0.95mm, F.Cu at (72.5, 76.3)
- added C9: 1uF, PCM_Capacitor_SMD_AKL:C_0603_1608Metric_Pad1.05x0.95mm, F.Cu at (82.3, 61.9)
- added RN3: 100 R_Array_Convex_4x1206, PCM_Resistor_SMD_AKL:R_Array_Concave_4x0603, F.Cu at (88.4, 81.7)
- added TP1: ~, ec_parts:PinHeader_1x04_P2.54mm_test_pad, F.Cu at (77.0, 54.7)
- added Y1: NX3215SA, PCM_Crystal_AKL:Crystal_SMD_3215-2Pin_3.2x1.5mm, F.Cu at (74.6, 75.9)
- C10: renamed from C16; footprint PCM_Capacitor_SMD_AKL:C_0603_1608Metric_Pad1.08x0.95mm -> PCM_Capacitor_SMD_AKL:C_0603_1608Metric_Pad1.05x0.95mm
- C2: footprint PCM_Capacitor_SMD_AKL:C_0603_1608Metric_Pad1.08x0.95mm -> PCM_Capacitor_SMD_AKL:C_0603_1608Metric_Pad1.05x0.95mm
- C3: renamed from C6; footprint PCM_Capacitor_SMD_AKL:C_0603_1608Metric_Pad1.08x0.95mm -> PCM_Capacitor_SMD_AKL:C_0603_1608Metric_Pad1.05x0.95mm
- C4: value 1uF -> 0.1uF; footprint PCM_Capacitor_SMD_AKL:C_0603_1608Metric_Pad1.08x0.95mm -> PCM_Capacitor_SMD_AKL:C_0603_1608Metric_Pad1.05x0.95mm
- C5: value ~ -> 4.7u; footprint PCM_Capacitor_SMD_AKL:C_0603_1608Metric_Pad1.08x0.95mm -> PCM_Capacitor_SMD_AKL:C_0603_1608Metric_Pad1.05x0.95mm
- C8: renamed from C3; footprint PCM_Capacitor_SMD_AKL:C_0603_1608Metric_Pad1.08x0.95mm -> PCM_Capacitor_SMD_AKL:C_0603_1608Metric_Pad1.05x0.95mm
- D1: footprint PCM_Diode_SMD_AKL:D_SOD-323F -> PCM_Diode_SMD_AKL:D_SOD-323_HandSoldering
- H1, H10, H11, H12, H2, H3, H4, H5, H6, H7, H8, H9: footprint MountingHole:MountingHole_2.1mm -> ec_parts:MountingHole_2.05mm
- RN1, RN2: value 4x0604 1k resistor array -> 1k R_Array_Concave_4x0603; footprint PCM_Resistor_SMD_AKL:R_Array_Convex_4x0612 -> PCM_Resistor_SMD_AKL:R_Array_Concave_4x0603
- SW1, SW10, SW11, SW12, SW13, SW14, SW15, SW16, SW17, SW18, SW19, SW2, SW20, SW21, SW22, SW23, SW24, SW25, SW26, SW27, SW28, SW3, SW4, SW5, SW6, SW7, SW8, SW9: value EC_SW -> ~
- SW29: value SW_Push -> PTS845
- U3: value nRF52840_holyiot_18010 -> DT1446-04S; footprint PCM_marbastlib-various:nRF52840_holyiot_18010_HS_simple -> PCM_Package_TO_SOT_SMD_AKL:SOT-363_SC-70-6_Handsoldering
- U5: value DT1446-04S -> STM32G0B1KETx; footprint PCM_Package_TO_SOT_SMD_AKL:SOT-363_SC-70-6_Handsoldering -> PCM_Package_QFP_AKL:LQFP-32_7x7mm_P0.8mm
- moved C5 48.8 mm to (73.9, 78.9), turned to 180 degrees
- moved U3 35.5 mm to (78.8, 51.0), turned to 0 degrees
- moved U5 27.5 mm to (81.2, 78.9)
- moved D1 27.4 mm to (85.5, 40.5), turned to 90 degrees
- moved H13 21.0 mm to (72.5, 96.0)
- moved C4 15.7 mm to (73.9, 80.6), turned to 180 degrees
- moved C2 14.6 mm to (77.3, 86.4)
- moved L1 14.2 mm to (86.5, 34.1), turned to 180 degrees
- moved U2 13.2 mm to (81.1, 90.1)
- moved R4 12.0 mm to (87.9, 40.2)
- moved J4 11.4 mm to (88.2, 68.3)
- moved C3 11.3 mm to (75.3, 101.4), turned to -90 degrees
- moved R6 11.2 mm to (77.3, 93.7), turned to -90 degrees
- moved U4 11.0 mm to (82.3, 58.9)
- moved C8 10.9 mm to (82.2, 55.9), turned to 180 degrees
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- renumbered H18 to H16, R4 to R2, R2 to R3, R5 to R4, R6 to R5, R9 to R6, R10 to R7
Connections:
- C10 pad 2: GNDA -> GND
- C2 pad 1: GNDA -> GND
- C3 pad 1: GNDA -> GND
- C5 pad 1: RESET -> +3V3
- C8 pad 1: VSYS -> +5V
- D1 pad 1: VSYS -> +5V
- D1 pad 2: +5V -> Net-(D1-A)
- F1 pad 1: Net-(D3-A) -> Net-(D1-A)
- H0 pad 1: GNDA -> GND
- H17 pad 1: USB_SHILED_2 -> GNDPWR
- J1 pad 1: SWDCLK -> +5V
- J1 pad 2: GND -> SWDIO
- J1 pad 3: SWDIO -> SWCLK
- J1 pad 4: +3V3 -> GND
- J2 pad R1: SCL -> USART_TX
- J2 pad R2: SDA -> USART_RX
- J3 pad S1: USB_SHILED_1 -> GNDPWR
- J3 pad S2: USB_SHILED_2 -> unconnected-(J3-SHIELD-PadS2)
- L1 pad 2: USB_SHILED_2 -> GNDPWR
- R4 pad 1: VBUS -> Net-(D1-A)
- R6 pad 2: GNDA -> GND
- RN1 pad 1: A2 -> A5
- RN1 pad 2: A1 -> A7
- RN1 pad 3: AO -> A6
- RN1 pad 4: A3 -> A4
- RN1 pad 5: GNDA -> GND
- RN1 pad 6: GNDA -> GND
- RN1 pad 7: GNDA -> GND
- RN1 pad 8: GNDA -> GND
- RN2 pad 1: RN1_1 -> AO
- RN2 pad 2: A6 -> A1
- RN2 pad 3: A7 -> A2
- RN2 pad 4: A5 -> RN1_4
- RN2 pad 5: GNDA -> GND
- RN2 pad 6: GNDA -> GND
- RN2 pad 7: GNDA -> GND
- RN2 pad 8: GNDA -> GND
- SW1 pad 1: A7 -> A1
- SW1 pad 3: GNDA -> GND
- SW10 pad 1: A3 -> A4
- SW10 pad 3: GNDA -> GND
- SW11 pad 1: AO -> A6
- SW11 pad 3: GNDA -> GND
- SW12 pad 1: AO -> A6
- SW12 pad 3: GNDA -> GND
- SW13 pad 1: AO -> A6
- SW13 pad 3: GNDA -> GND
- SW14 pad 1: A1 -> A7
- SW14 pad 3: GNDA -> GND
- SW15 pad 1: A1 -> A7
- SW15 pad 3: GNDA -> GND
- SW16 pad 1: A1 -> A7
- SW16 pad 3: GNDA -> GND
- SW17 pad 1: A2 -> A5
- SW17 pad 3: GNDA -> GND
- SW18 pad 1: A2 -> A5
- SW18 pad 3: GNDA -> GND
- SW19 pad 1: A2 -> A5
- SW19 pad 3: GNDA -> GND
- SW2 pad 1: A7 -> A1
- SW2 pad 3: GNDA -> GND
- SW20 pad 1: A5 -> A2
- SW20 pad 3: GNDA -> GND
- SW21 pad 1: A5 -> A2
- SW21 pad 3: GNDA -> GND
- SW22 pad 1: A5 -> A2
- SW22 pad 3: GNDA -> GND
- SW23 pad 1: A6 -> AO
- SW23 pad 3: GNDA -> GND
- SW24 pad 1: A3 -> A4
- SW24 pad 3: GNDA -> GND
- SW25 pad 1: AO -> A6
- SW25 pad 3: GNDA -> GND
- SW26 pad 1: A1 -> A7
- SW26 pad 3: GNDA -> GND
- SW27 pad 1: A2 -> A5
- SW27 pad 3: GNDA -> GND
- SW28 pad 1: A5 -> A2
- SW28 pad 3: GNDA -> GND
- SW29 pad 2: RESET -> /NRST
- SW3 pad 1: A7 -> A1
- SW3 pad 3: GNDA -> GND
- SW4 pad 1: A7 -> A1
- SW4 pad 3: GNDA -> GND
- SW5 pad 1: A6 -> AO
- SW5 pad 3: GNDA -> GND
- SW6 pad 1: A6 -> AO
- SW6 pad 3: GNDA -> GND
- SW7 pad 1: A6 -> AO
- SW7 pad 3: GNDA -> GND
- SW8 pad 1: A3 -> A4
- SW8 pad 3: GNDA -> GND
- SW9 pad 1: A3 -> A4
- SW9 pad 3: GNDA -> GND
- U1 pad 7: GNDA -> GND
- U1 pad 8: GNDA -> GND
- U2 pad 4: GNDA -> GND
- U3 pad 1: GND -> USART_RX
- U3 pad 2: unconnected-(U3-P1.11-LF-Pad2) -> GND
- U3 pad 3: unconnected-(U3-P1.10-LF-Pad3) -> D+
- U3 pad 4: unconnected-(U3-P1.13-LF-Pad4) -> D-
- U3 pad 5: unconnected-(U3-P1.15-LF-Pad5) -> +5V
- U3 pad 6: ADC -> USART_TX
- U4 pad 1: VSYS -> +5V
- U4 pad 3: VSYS -> +5V
- U5 pad 1: SCL -> USART_RX
- U5 pad 2: GND -> /OSC32_IN
- U5 pad 3: SDA -> /OSC32_OUT
- U5 pad 4: VBUS_DEC -> +3V3
- U5 pad 5: +5V -> GND
- U5 pad 6: unconnected-(U5-IO4-Pad6) -> /NRST
Routing:
- net A4: track 0.00 -> 136.1 mm, vias 0 -> 5
- net A3: track 134.5 -> 0.00 mm, vias 5 -> 0
- net A1: track 99.9 -> 191.4 mm
- net A7: track 190.9 -> 102.1 mm
- net RESET: track 60.8 -> 0.00 mm, vias 2 -> 0
- net /NRST: track 0.00 -> 56.3 mm, vias 0 -> 2
- net +3V3: track 112.1 -> 68.9 mm, vias 8 -> 5
- net SCL: track 42.5 -> 0.00 mm
- net AO: track 117.7 -> 160.2 mm
- net SDA: track 41.7 -> 0.00 mm
- net USART_TX: track 0.00 -> 41.2 mm, vias 0 -> 2
- net USART_RX: track 0.00 -> 40.8 mm
- net A6: track 160.1 -> 119.6 mm
- net +5V: track 68.5 -> 38.3 mm, vias 3 -> 2
- net VBAT: track 29.0 -> 0.00 mm, vias 2 -> 0
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- removed copper zone on B.Cu, net GNDA
- removed copper zone on F.Cu, net GNDA
Other:
- board text added: "VCC"
- board text removed: "+"
- board text removed: "+3.3V"
- board text removed: "-"

Commit message: Fix capacitor, resistor values
Parts:
- C6, C7: value 5.6p -> 22p
- RN3: value 100 R_Array_Convex_4x1206 -> 100 R_Array_Convex_4x0603
- Y1: value NX3215SA -> 32.768kHz
Changed lines of the file:
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@@
   (title_block
     (title "Corne EEC")
-    (date "2023-06-22")
+    (date "2023-07-18")
     (rev "1.0")
     (comment 1 "Copyright © 2023")
@@
         (effects (font (size 1 1) (thickness 0.15)))
     )
-    (fp_text value "100 R_Array_Convex_4x1206" (at 0 2.6) (layer "F.Fab") hide
+    (fp_text value "100 R_Array_Convex_4x0603" (at 0 2.6) (layer "F.Fab") hide
         (effects (font (size 1 1) (thickness 0.15)))
     )
@@
         (effects (font (size 1 1) (thickness 0.15)))
     )
-    (fp_text value "NX3215SA" (at 0 2 90) (layer "F.Fab") hide
+    (fp_text value "32.768kHz " (at 0 2 90) (layer "F.Fab") hide
         (effects (font (size 1 1) (thickness 0.15)))
     )
@@
         (effects (font (size 1 1) (thickness 0.15)))
     )
-    (fp_text value "5.6p" (at 0 1.43 90) (layer "F.Fab") hide
+    (fp_text value "22p" (at 0 1.43 90) (layer "F.Fab") hide
         (effects (font (size 1 1) (thickness 0.15)))
     )
@@
         (effects (font (size 1 1) (thickness 0.15)))
     )
-    (fp_text value "5.6p" (at 0 1.43) (layer "F.Fab") hide
+    (fp_text value "22p" (at 0 1.43) (layer "F.Fab") hide
         (effects (font (size 1 1) (thickness 0.15)))
     )
