File: hardware/pcb/keyboard/keyboard_left.kicad_sch (KiCad schematic)
At the start: 37 parts, among them J1 SM04B-SRSS-TB, J2 PJ320D, J3 HRO_TYPE-C-31-M-12, J4 FH34SRJ-12S-0.5SH, SW29 PTS845, U3 DT1446-04S, U4 XC6220B331MR-G, U5 STM32G431KBTx, U6 CH334R, Y1 8MHz, Y2 8MHz

Commit message: preproduction
Parts:
- removed U3: DT1446-04S, PCM_Package_TO_SOT_SMD_AKL:SOT-363_SC-70-6_Handsoldering, symbol Power_Protection:SRV05-4
- added U3: PRTR5V0U2X, PCM_Package_TO_SOT_SMD_AKL:SOT-143, symbol Power_Protection:PRTR5V0U2X
- C12, C13, C6, C7: value 22p -> 10pF
- Y2: value 8MHz -> 12MHz
Connections:
- net +5V: now also U3.4 (VCC)
- net GND: now also U3.1 (GND)
- net UP_D+: now also U3.3 (I/O2)
- net UP_D-: now also U3.2 (I/O1)
Changed lines of the file:
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@@
     (stroke (width 0) (type default))
   )
-  (wire (pts (xy 270.51 41.91) (xy 273.05 41.91))
-    (stroke (width 0) (type default))
-  )
   (wire (pts (xy 171.45 25.4) (xy 168.91 25.4))
     (stroke (width 0) (type default))
@@
     (effects (font (size 1.27 1.27)) (justify left bottom))
   )
+  (label "UP_D+" (at 152.4 138.43 0) (fields_autoplaced)
+    (effects (font (size 1.27 1.27)) (justify left bottom))
+  )
   (label "DM4" (at 182.88 106.68 180) (fields_autoplaced)
     (effects (font (size 1.27 1.27)) (justify right bottom))
@@
     (effects (font (size 1.27 1.27)) (justify left bottom))
   )
-  (label "UP_D+" (at 152.4 140.97 0) (fields_autoplaced)
-    (effects (font (size 1.27 1.27)) (justify left bottom))
-  )
   (label "MCU_D+" (at 25.4 110.49 180) (fields_autoplaced)
     (effects (font (size 1.27 1.27)) (justify right bottom))
@@
     (effects (font (size 1.27 1.27)) (justify left bottom))
   )
-  (label "UP_D-" (at 152.4 135.89 0) (fields_autoplaced)
-    (effects (font (size 1.27 1.27)) (justify left bottom))
-  )
   (label "ADC12_IN1" (at 198.12 38.1 0) (fields_autoplaced)
     (effects (font (size 1.27 1.27)) (justify left bottom))
@@
     (effects (font (size 1.27 1.27)) (justify right bottom))
   )
+  (label "UP_D-" (at 127 138.43 180) (fields_autoplaced)
+    (effects (font (size 1.27 1.27)) (justify right bottom))
+  )
   (label "VDDA" (at 140.97 80.01 0) (fields_autoplaced)
     (effects (font (size 1.27 1.27)) (justify left bottom))
@@
     )
   )
-  (global_label "USART_TX" (shape input) (at 127 140.97 180) (fields_autoplaced)
-    (effects (font (size 1.27 1.27)) (justify right))
-    (property "Intersheetrefs" "${INTERSHEET_REFS}" (at 116.3352 140.97 0)
-      (effects (font (size 1.27 1.27)) (justify right) hide)
-    )
-  )
   (global_label "AO" (shape input) (at 273.05 34.29 0) (fields_autoplaced)
     (effects (font (size 1.27 1.27)) (justify left))
@@
     )
   )
-  (global_label "USART_RX" (shape input) (at 127 135.89 180) (fields_autoplaced)
-    (effects (font (size 1.27 1.27)) (justify right))
-    (property "Intersheetrefs" "${INTERSHEET_REFS}" (at 116.3352 135.89 0)
-      (effects (font (size 1.27 1.27)) (justify right) hide)
-    )
-  )
   (global_label "COL4" (shape input) (at 270.51 34.29 180) (fields_autoplaced)
     (effects (font (size 1.27 1.27)) (justify right))
@@
       (effects (font (size 1.27 1.27)))
     )
-    (property "Value" "22p" (at 59.69 76.2 0)
+    (property "Value" "10pF" (at 59.69 76.2 0)
       (effects (font (size 1.27 1.27)))
     )
@@
       (effects (font (size 1.27 1.27)))
     )
-    (property "Value" "8MHz" (at 53.34 81.28 90)
+    (property "Value" "12MHz" (at 53.34 81.28 90)
       (effects (font (size 1.27 1.27)))
     )
@@
       (effects (font (size 1.27 1.27)))
     )
-    (property "Value" "22p" (at 125.73 54.61 90)
+    (property "Value" "10pF" (at 125.73 54.61 90)
       (effects (font (size 1.27 1.27)))
     )
@@
       (effects (font (size 1.27 1.27)))
     )
-    (property "Value" "22p" (at 44.45 76.2 0)
+    (property "Value" "10pF" (at 44.45 76.2 0)
       (effects (font (size 1.27 1.27)))
     )
@@
     )
   )
+  (symbol (lib_id "power:GND") (at 273.05 41.91 270) (mirror x) (unit 1)
+    (in_bom yes) (on_board yes) (dnp no)
+    (property "Reference" "#PWR052" (at 266.7 41.91 0)
+      (effects (font (size 1.27 1.27)) hide)
+    )
+    (property "Value" "GND" (at 269.24 41.91 90)
+      (effects (font (size 1.27 1.27)) (justify right))
+    )
+    (property "Footprint" "" (at 273.05 41.91 0)
+      (effects (font (size 1.27 1.27)) hide)
+    )
+    (property "Datasheet" "" (at 273.05 41.91 0)
+      (effects (font (size 1.27 1.27)) hide)
+    )
+    (pin "1")
+    (instances
+      (project "keyboard_left"
+        (path "/852dabbf-de45-4470-8176-59d37a754407"
+          (reference "#PWR052") (unit 1)
+        )
+      )
+      (project "EC60-Rev_1_1"
+        (path "/e63e39d7-6ac0-4ffd-8aa3-1841a4541b55"
+          (reference "#PWR020") (unit 1)
+        )
+      )
+    )
+  )
+  (symbol (lib_id "Power_Protection:PRTR5V0U2X") (at 139.7 138.43 0) (unit 1)
+    (in_bom yes) (on_board yes) (dnp no)
+    (property "Reference" "U3" (at 149.86 129.54 0)
+      (effects (font (size 1.27 1.27)))
+    )
+    (property "Value" "PRTR5V0U2X" (at 153.67 132.08 0)
+      (effects (font (size 1.27 1.27)))
+    )
+    (property "Footprint" "PCM_Package_TO_SOT_SMD_AKL:SOT-143" (at 141.224 138.43 0)
+      (effects (font (size 1.27 1.27)) hide)
+    )
+    (property "Datasheet" "https://assets.nexperia.com/documents/data-sheet/PRTR5V0U2X.pdf" (at 141.224 138.43 0)
+      (effects (font (size 1.27 1.27)) hide)
+    )
+    (property "LCSC" "C2827688" (at 139.7 138.43 0)
+      (effects (font (size 1.27 1.27)) hide)
+    )
+    (pin "1")
+    (pin "2")
+    (pin "3")
+    (pin "4")
+    (instances
+      (project "keyboard_left"
+        (path "/852dabbf-de45-4470-8176-59d37a754407"
+          (reference "U3") (unit 1)
+        )
+      )
+      (project "EC60-Rev_1_1"
+        (path "/e63e39d7-6ac0-4ffd-8aa3-1841a4541b55"
+          (reference "D1") (unit 1)
+        )
+      )
+    )
+  )
   (symbol (lib_id "power:VBUS") (at 69.85 102.87 270) (unit 1)
     (in_bom yes) (on_board yes) (dnp no)
@@
     )
   )
-  (symbol (lib_id "power:GNDA") (at 270.51 41.91 270) (unit 1)
-    (in_bom yes) (on_board yes) (dnp no)
-    (property "Reference" "#PWR052" (at 264.16 41.91 0)
-      (effects (font (size 1.27 1.27)) hide)
-    )
-    (property "Value" "GNDA" (at 266.7 41.91 90)
-      (effects (font (size 1.27 1.27)) (justify right))
-    )
-    (property "Footprint" "" (at 270.51 41.91 0)
-      (effects (font (size 1.27 1.27)) hide)
-    )
-    (property "Datasheet" "" (at 270.51 41.91 0)
-      (effects (font (size 1.27 1.27)) hide)
-    )
-    (pin "1")
-    (instances
-      (project "keyboard_left"
-        (path "/852dabbf-de45-4470-8176-59d37a754407"
-          (reference "#PWR052") (unit 1)
-        )
-        (path "/852dabbf-de45-4470-8176-59d37a754407/ac97752b-a16f-44ee-ad7e-0bcdbcea7979"
-          (reference "#PWR043") (unit 1)
-        )
-      )
-    )
-  )
   (symbol (lib_id "nrfmicro-rescue:GND") (at 154.94 104.14 90) (unit 1)
     (in_bom yes) (on_board yes) (dnp no)
@@
       (effects (font (size 1.27 1.27)))
     )
-    (property "Value" "22p" (at 124.46 41.91 90)
+    (property "Value" "10pF" (at 124.46 41.91 90)
       (effects (font (size 1.27 1.27)))
     )
@@
         )
       )
-    )
-  )
-  (symbol (lib_id "Power_Protection:SRV05-4") (at 139.7 138.43 0) (unit 1)
-    (in_bom yes) (on_board yes) (dnp no) (fields_autoplaced)
-    (property "Reference" "U3" (at 142.8497 124.46 0)
-      (effects (font (size 1.27 1.27)) (justify left))
-    )
-    (property "Value" "DT1446-04S" (at 142.8497 127 0)
-      (effects (font (size 1.27 1.27)) (justify left))
-    )
-    (property "Footprint" "PCM_Package_TO_SOT_SMD_AKL:SOT-363_SC-70-6_Handsoldering" (at 157.48 149.86 0)
-      (effects (font (size 1.27 1.27)) hide)
-    )
-    (property "Datasheet" "http://www.onsemi.com/pub/Collateral/SRV05-4-D.PDF" (at 139.7 138.43 0)
-      (effects (font (size 1.27 1.27)) hide)
-    )
-    (property "Comment" "" (at 139.7 138.43 0)
-      (effects (font (size 1.27 1.27)) hide)
-    )
-    (pin "1")
-    (pin "2")
-    (pin "3")
-    (pin "4")
-    (pin "5")
-    (pin "6")
-    (instances
-      (project "keyboard_left"
-        (path "/852dabbf-de45-4470-8176-59d37a754407"
-          (reference "U3") (unit 1)
-        )
-      )
