File: hardware/pcb/keyboard/keyboard_left.kicad_sch (KiCad schematic)
At the start: 34 parts, among them J1 SM03B-SRSS-TB, J2 PJ320D, J3 HRO_TYPE-C-31-M-12, J4 HRS_FH34SRJ-06S-0.5SH(50), SW29 PTS845, U3 PRTR5V0U2X, U4 XC6220B331MR-G, U5 STM32G431KBTx, U6 24FC01T-I/OT, Y1 24MHz 10pF

Commit message: back
Parts:
- Y1: value 24MHz 10pF -> 8MHz 10pF
Changed lines of the file:
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@@
 			)
 		)
-		(property "Value" "24MHz 10pF"
+		(property "Value" "8MHz 10pF"
 			(at 135.89 49.53 90)
 			(effects

Commit message: Generate production files.
Parts:
- D1: value 1N5819 -> BAT60B; Comment (none) -> Alternative: 1N5819
- U4: Comment (none) -> Alternative: AP2112K
Changed lines of the file:
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@@
 	(title_block
 		(title "Corne EEC - Keyboard Left")
-		(date "2025-08-31")
+		(date "2025-09-18")
 		(rev "2.0")
 		(company "https://github.com/daehyeok/Corne_EEC")
@@
 			)
 		)
-		(property "Value" "1N5819"
+		(property "Value" "BAT60B"
 			(at 66.3575 27.94 0)
 			(effects
@@
 			)
 		)
-		(property "Comment" ""
+		(property "Comment" "Alternative: 1N5819"
 			(at 66.04 31.75 0)
 			(effects
@@
 			)
 		)
-		(property "Comment" ""
+		(property "Comment" "Alternative: AP2112K"
 			(at 92.71 34.29 0)
 			(effects

Commit message: Rev 2.1
Parts:
- D1: value BAT60B -> 1N5819; Comment Alternative: 1N5819 -> (none)
- J4: footprint ec_parts:CONN6x1_FH34SRJ-6S-0.5SH50_HIR -> ec_parts:CONN6x1_FH12S-6S-1SH55
- U4: Comment Alternative: AP2112K -> (none)
Changed lines of the file:
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@@
 	(title_block
 		(title "Corne EEC - Keyboard Left")
-		(date "2025-09-18")
+		(date "2025-08-31")
 		(rev "2.0")
 		(company "https://github.com/daehyeok/Corne_EEC")
@@
 			)
 		)
-		(property "Value" "BAT60B"
+		(property "Value" "1N5819"
 			(at 66.3575 27.94 0)
 			(effects
@@
 			)
 		)
-		(property "Comment" "Alternative: 1N5819"
+		(property "Comment" ""
 			(at 66.04 31.75 0)
 			(effects
@@
 			)
 		)
-		(property "Footprint" "ec_parts:CONN6x1_FH34SRJ-6S-0.5SH50_HIR"
+		(property "Footprint" "ec_parts:CONN6x1_FH12S-6S-1SH55"
 			(at 196.85 119.38 0)
 			(effects
@@
 			)
 		)
-		(property "Comment" "Alternative: AP2112K"
+		(property "Comment" ""
 			(at 92.71 34.29 0)
 			(effects
