File: hardware/pcb/keyboard/key_matrix.kicad_sch (KiCad schematic)
At the start: 82 parts, among them U1 74HC4051, U2 OPA350UA

Commit message: temp
Parts:
- C16, C2, C6: footprint PCM_Capacitor_SMD_AKL:C_0603_1608Metric_Pad1.05x0.95mm -> PCM_Capacitor_SMD_AKL:C_0603_1608Metric
- R10, R9: footprint PCM_Resistor_SMD_AKL:R_0603_1608Metric_Pad0.98x0.95mm -> PCM_Resistor_SMD_AKL:R_0603_1608Metric

Commit message: temp
Parts:
- RN1, RN2: renamed from RN?; value 1k R_Array_Concave_4x0603 -> 100k R_Array_Concave_4x0603

Commit message: rev2
Parts:
- renumbered C16 to C10, C6 to C2, C2 to C3, G27 to G28, H1 to H0, H2 to H10, H2 to H11, H2 to H12, H2 to H13, H2 to H14, H2 to H15, H2 to H16, H2 to H3, H2 to H4, H2 to H5, H2 to H6, H2 to H7, H2 to H8, H2 to H9, R9 to R6, R10 to R7, SW20 to SW28
Changed lines of the file:
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@@
 (kicad_sch
-	(version 20231120)
+	(version 20250114)
 	(generator "eeschema")
-	(generator_version "8.0")
+	(generator_version "9.0")
 	(paper "A4")
 	(title_block
@@
 		(comment 2 "MIT License")
 	)
+	(rectangle
+		(start 195.58 20.32)
+		(end 283.21 62.23)
+		(stroke
+			(width 0)
+			(type default)
+		)
+		(fill
+			(type none)
+		)
+	)
+	(rectangle
+		(start 19.05 114.3)
+		(end 156.21 180.34)
+		(stroke
+			(width 0)
+			(type default)
+		)
+		(fill
+			(type none)
+		)
+	)
+	(rectangle
+		(start 19.05 20.32)
+		(end 193.04 109.22)
+		(stroke
+			(width 0)
+			(type default)
+		)
+		(fill
+			(type none)
+		)
+	)
+	(rectangle
+		(start 195.58 64.77)
+		(end 281.94 109.22)
+		(stroke
+			(width 0)
+			(type default)
+		)
+		(fill
+			(type none)
+		)
+	)
+	(text "Analog Sensing circuit\n"
+		(exclude_from_sim no)
+		(at 20.32 116.84 0)
+		(effects
+			(font
+				(size 1.27 1.27)
+			)
+			(justify left bottom)
+		)
+	)
+	(text "EC Switch Matrix\n"
+		(exclude_from_sim no)
+		(at 22.86 24.13 0)
+		(effects
+			(font
+				(size 1.27 1.27)
+			)
+			(justify left bottom)
+		)
+	)
+	(text "NOTE:\n- in order to controll the output of the sensing circuit you can change\nthe value of R7 to fit a higer/lower gain of the OpAmp.\n"
+		(exclude_from_sim no)
+		(at 20.32 175.26 0)
+		(effects
+			(font
+				(size 1.27 1.27)
+			)
+			(justify left bottom)
+		)
+	)
+	(text "H1~H7 - For pcb and plate"
+		(exclude_from_sim no)
+		(at 201.93 83.82 0)
+		(effects
+			(font
+				(size 1.27 1.27)
+			)
+			(justify left bottom)
+		)
+	)
+	(text "H8~12 located on board edge for top case(Optional)"
+		(exclude_from_sim no)
+		(at 201.93 92.71 0)
+		(effects
+			(font
+				(size 1.27 1.27)
+			)
+			(justify left bottom)
+		)
+	)
+	(text "Dummy footprints to draw housing/keycap area on user comment and drawing layer.\n"
+		(exclude_from_sim no)
+		(at 198.12 24.13 0)
+		(effects
+			(font
+				(size 1.27 1.27)
+			)
+			(justify left bottom)
+		)
+	)
+	(text "M1.6 Mounting Holes for doughter board."
+		(exclude_from_sim no)
+		(at 196.85 101.6 0)
+		(effects
+			(font
+				(size 1.27 1.27)
+			)
+			(justify left bottom)
+		)
+	)
+	(text "M2 Mounting Holes "
+		(exclude_from_sim no)
+		(at 196.85 80.01 0)
+		(effects
+			(font
+				(size 1.27 1.27)
+			)
+			(justify left bottom)
+		)
+	)
+	(text "Optional GND connector/M1.6 Mount"
+		(exclude_from_sim no)
+		(at 196.85 68.58 0)
+		(effects
+			(font
+				(size 1.27 1.27)
+			)
+			(justify left bottom)
+		)
+	)
 	(junction
 		(at 132.08 63.5)
@@
 		)
 	)
-	(rectangle
-		(start 195.58 20.32)
-		(end 283.21 62.23)
-		(stroke
-			(width 0)
-			(type default)
-		)
-		(fill
-			(type none)
-		)
-	)
-	(rectangle
-		(start 19.05 114.3)
-		(end 156.21 180.34)
-		(stroke
-			(width 0)
-			(type default)
-		)
-		(fill
-			(type none)
-		)
-	)
-	(rectangle
-		(start 19.05 20.32)
-		(end 193.04 109.22)
-		(stroke
-			(width 0)
-			(type default)
-		)
-		(fill
-			(type none)
-		)
-	)
-	(rectangle
-		(start 195.58 64.77)
-		(end 281.94 109.22)
-		(stroke
-			(width 0)
-			(type default)
-		)
-		(fill
-			(type none)
-		)
-	)
-	(text "Analog Sensing circuit\n"
-		(exclude_from_sim no)
-		(at 20.32 116.84 0)
-		(effects
-			(font
-				(size 1.27 1.27)
-			)
-			(justify left bottom)
-		)
-	)
-	(text "EC Switch Matrix\n"
-		(exclude_from_sim no)
-		(at 22.86 24.13 0)
-		(effects
-			(font
-				(size 1.27 1.27)
-			)
-			(justify left bottom)
-		)
-	)
-	(text "NOTE:\n- in order to controll the output of the sensing circuit you can change\nthe value of R7 to fit a higer/lower gain of the OpAmp.\n"
-		(exclude_from_sim no)
-		(at 20.32 175.26 0)
-		(effects
-			(font
-				(size 1.27 1.27)
-			)
-			(justify left bottom)
-		)
-	)
-	(text "H1~H7 - For pcb and plate"
-		(exclude_from_sim no)
-		(at 201.93 83.82 0)
-		(effects
-			(font
-				(size 1.27 1.27)
-			)
-			(justify left bottom)
-		)
-	)
-	(text "H8~12 located on board edge for top case(Optional)"
-		(exclude_from_sim no)
-		(at 201.93 92.71 0)
-		(effects
-			(font
-				(size 1.27 1.27)
-			)
-			(justify left bottom)
-		)
-	)
-	(text "Dummy footprints to draw housing/keycap area on user comment and drawing layer.\n"
-		(exclude_from_sim no)
-		(at 198.12 24.13 0)
-		(effects
-			(font
-				(size 1.27 1.27)
-			)
-			(justify left bottom)
-		)
-	)
-	(text "M1.6 Mounting Holes for doughter board."
-		(exclude_from_sim no)
-		(at 196.85 101.6 0)
-		(effects
-			(font
-				(size 1.27 1.27)
-			)
-			(justify left bottom)
-		)
-	)
-	(text "M2 Mounting Holes "
-		(exclude_from_sim no)
-		(at 196.85 80.01 0)
-		(effects
-			(font
-				(size 1.27 1.27)
-			)
-			(justify left bottom)
-		)
-	)
-	(text "Optional GND connector/M1.6 Mount"
-		(exclude_from_sim no)
-		(at 196.85 68.58 0)
-		(effects
-			(font
-				(size 1.27 1.27)
-			)
-			(justify left bottom)
-		)
-	)
 	(global_label "RN0_3"
 		(shape input)
@@
 		(on_board yes)
 		(dnp no)
-		(property "Reference" "R9"
+		(property "Reference" "R6"
 			(at 116.84 151.13 0)
 			(effects
@@
 		(dnp no)
 		(fields_autoplaced yes)
-		(property "Reference" "H2"
+		(property "Reference" "H14"
 			(at 213.36 105.4099 0)
 			(effects
@@
 		(dnp no)
 		(fields_autoplaced yes)
-		(property "Reference" "H2"
+		(property "Reference" "H9"
 			(at 237.49 95.2499 0)
 			(effects
@@
 		(dnp no)
 		(fields_autoplaced yes)
-		(property "Reference" "H2"
+		(property "Reference" "H3"
 			(at 214.63 95.2499 0)
 			(effects
@@
 		(on_board yes)
 		(dnp no)
-		(property "Reference" "C2"
+		(property "Reference" "C3"
 			(at 144.78 157.5308 90)
 			(effects
@@
 		(dnp no)
 		(fields_autoplaced yes)
-		(property "Reference" "H2"
+		(property "Reference" "H11"
 			(at 245.11 86.3599 0)
 			(effects
@@
 		(dnp no)
 		(fields_autoplaced yes)
-		(property "Reference" "H2"
+		(property "Reference" "H7"
 			(at 229.87 95.2499 0)
 			(effects
@@
 		(dnp no)
 		(fields_autoplaced yes)
-		(property "Reference" "H2"
+		(property "Reference" "H12"
 			(at 252.73 86.3599 0)
 			(effects
@@
 		(dnp no)
 		(fields_autoplaced yes)
-		(property "Reference" "H2"
+		(property "Reference" "H6"
 			(at 222.25 86.3599 0)
 			(effects
@@
 		(on_board yes)
 		(dnp no)
-		(property "Reference" "H1"
+		(property "Reference" "H0"
 			(at 210.82 72.39 90)
 			(effects
@@
 		(on_board yes)
 		(dnp no)
-		(property "Reference" "R10"
+		(property "Reference" "R7"
 			(at 126.365 146.05 90)
 			(effects
@@
 		(dnp no)
 		(fields_autoplaced yes)
-		(property "Reference" "H2"
+		(property "Reference" "H5"
 			(at 222.25 95.2499 0)
 			(effects
@@
 		(dnp no)
 		(fields_autoplaced yes)
-		(property "Reference" "H2"
+		(property "Reference" "H4"
 			(at 214.63 86.3599 0)
 			(effects
@@
 		(dnp no)
 		(fields_autoplaced yes)
-		(property "Reference" "SW20"
+		(property "Reference" "SW28"
 			(at 172.72 33.2445 0)
 			(effects
@@
 		(dnp no)
 		(fields_autoplaced yes)
-		(property "Reference" "H2"
+		(property "Reference" "H15"
 			(at 220.98 105.4099 0)
 			(effects
@@
 		(on_board yes)
 		(dnp no)
-		(property "Reference" "C6"
+		(property "Reference" "C2"
 			(at 78.74 116.7892 90)
 			(effects
@@
 		(on_board yes)
 		(dnp no)
-		(property "Reference" "H2"
+		(property "Reference" "H16"
 			(at 228.6 105.4099 0)
 			(effects
@@
 		(dnp no)
 		(fields_autoplaced yes)
-		(property "Reference" "G27"
+		(property "Reference" "G28"
 			(at 274.32 31.7499 0)
 			(effects
@@
 		(dnp no)
 		(fields_autoplaced yes)
-		(property "Reference" "H2"
+		(property "Reference" "H8"
 			(at 229.87 86.3599 0)
 			(effects
@@
 		(dnp no)
 		(fields_autoplaced yes)
-		(property "Reference" "H2"
+		(property "Reference" "H10"
 			(at 237.49 86.3599 0)
 			(effects
@@
 		(on_board yes)
 		(dnp no)
-		(property "Reference" "C16"
+		(property "Reference" "C10"
 			(at 97.7392 138.43 90)
 			(effects
@@
 		(dnp no)
 		(fields_autoplaced yes)
-		(property "Reference" "H2"
+		(property "Reference" "H13"
 			(at 205.74 105.4099 0)
 			(effects

Commit message: init memory
Parts:
- added H18, H19: ~, ec_parts:SMT-SO-M1.6-screwhole_only, symbol Mechanical:MountingHole
Changed lines of the file:
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@@
 	(symbol
 		(lib_id "Mechanical:MountingHole")
+		(at 234.95 105.41 0)
+		(unit 1)
+		(exclude_from_sim no)
+		(in_bom yes)
+		(on_board yes)
+		(dnp no)
+		(fields_autoplaced yes)
+		(property "Reference" "H18"
+			(at 237.49 105.4099 0)
+			(effects
+				(font
+					(size 1.27 1.27)
+				)
+				(justify left)
+			)
+		)
+		(property "Value" "~"
+			(at 237.49 106.6799 0)
+			(effects
+				(font
+					(size 1.27 1.27)
+				)
+				(justify left)
+			)
+		)
+		(property "Footprint" "ec_parts:SMT-SO-M1.6-screwhole_only"
+			(at 234.95 105.41 0)
+			(effects
+				(font
+					(size 1.27 1.27)
+				)
+				(hide yes)
+			)
+		)
+		(property "Datasheet" "~"
+			(at 234.95 105.41 0)
+			(effects
+				(font
+					(size 1.27 1.27)
+				)
+				(hide yes)
+			)
+		)
+		(property "Description" ""
+			(at 234.95 105.41 0)
+			(effects
+				(font
+					(size 1.27 1.27)
+				)
+				(hide yes)
+			)
+		)
+		(property "Field4" ""
+			(at 234.95 105.41 0)
+			(effects
+				(font
+					(size 1.27 1.27)
+				)
+				(hide yes)
+			)
+		)
+		(property "Comment" ""
+			(at 234.95 105.41 0)
+			(effects
+				(font
+					(size 1.27 1.27)
+				)
+				(hide yes)
+			)
+		)
+		(instances
+			(project "keyboard_left"
+				(path "/852dabbf-de45-4470-8176-59d37a754407/ac97752b-a16f-44ee-ad7e-0bcdbcea7979"
+					(reference "H18")
+					(unit 1)
+				)
+			)
+		)
+	)
+	(symbol
+		(lib_id "Mechanical:MountingHole")
 		(at 212.09 95.25 0)
 		(unit 1)
@@
 					(unit 1)
 				)
+			)
+		)
+	)
+	(symbol
+		(lib_id "Mechanical:MountingHole")
+		(at 242.57 105.41 0)
+		(unit 1)
+		(exclude_from_sim no)
+		(in_bom yes)
+		(on_board yes)
+		(dnp no)
+		(property "Reference" "H19"
+			(at 245.11 105.4099 0)
+			(effects
+				(font
+					(size 1.27 1.27)
+				)
+				(justify left)
+			)
+		)
+		(property "Value" "~"
+			(at 245.11 106.6799 0)
+			(effects
+				(font
+					(size 1.27 1.27)
+				)
+				(justify left)
+			)
+		)
+		(property "Footprint" "ec_parts:SMT-SO-M1.6-screwhole_only"
+			(at 242.57 105.41 0)
+			(effects
+				(font
+					(size 1.27 1.27)
+				)
+				(hide yes)
+			)
+		)
+		(property "Datasheet" "~"
+			(at 242.57 105.41 0)
+			(effects
+				(font
+					(size 1.27 1.27)
+				)
+				(hide yes)
+			)
+		)
+		(property "Description" ""
+			(at 242.57 105.41 0)
+			(effects
+				(font
+					(size 1.27 1.27)
+				)
+				(hide yes)
+			)
+		)
+		(property "Field4" ""
+			(at 242.57 105.41 0)
+			(effects
+				(font
+					(size 1.27 1.27)
+				)
+				(hide yes)
+			)
+		)
+		(property "Comment" ""
+			(at 242.57 105.41 0)
+			(effects
+				(font
+					(size 1.27 1.27)
+				)
+				(hide yes)
+			)
+		)
+		(instances
+			(project "keyboard_left"
+				(path "/852dabbf-de45-4470-8176-59d37a754407/ac97752b-a16f-44ee-ad7e-0bcdbcea7979"
+					(reference "H19")
+					(unit 1)
+				)

Commit message: update schema.
Other:
- company: (none) -> https://github.com/daehyeok/Corne_EEC
Changed lines of the file:
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@@
 	(title_block
 		(title "Key Matrix")
-		(date "2023-07-18")
+		(date "2025-08-31")
 		(rev "1.0")
+		(company "https://github.com/daehyeok/Corne_EEC")
 		(comment 2 "MIT License")
 	)
