File: hardware/pcb/keyboard/keyboard_right.kicad_sch (KiCad schematic)
At the start: 35 parts, among them J1 SM04B-SRSS-TB, J2 PJ320D, J3 HRO_TYPE-C-31-M-12, J4 HRS_FH34SRJ-06S-0.5SH(50), SW29 PTS845, U3 PRTR5V0U2X, U4 XC6220B331MR-G, U5 STM32G431KBTx, U6 24FC01T-I/OT, Y1 8MHz 10pF

Commit message: Generate production files.
Parts:
- D1: value 1N5819 -> BAT60B; Comment (none) -> Alternative: 1N5819
- U4: Comment (none) -> Alternative: AP2112K
Changed lines of the file:
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@@
 	(title_block
 		(title "Corne EEC - Keyboard Right")
-		(date "2025-08-31")
+		(date "2025-09-18")
 		(rev "2.0")
 		(company "https://github.com/daehyeok/Corne_EEC")
@@
 	)
 	(junction
-		(at 95.25 128.27)
-		(diameter 0)
-		(color 0 0 0 0)
-	)
-	(junction
 		(at 82.55 118.11)
 		(diameter 0)
@@
 	)
 	(junction
-		(at 179.07 83.82)
+		(at 72.39 118.11)
 		(diameter 0)
 		(color 0 0 0 0)
 	)
 	(junction
-		(at 72.39 118.11)
+		(at 179.07 83.82)
 		(diameter 0)
 		(color 0 0 0 0)
@@
 	)
 	(junction
+		(at 95.25 128.27)
+		(diameter 0)
+		(color 0 0 0 0)
+	)
+	(junction
 		(at 52.07 123.19)
 		(diameter 0)
@@
 					(size 1.27 1.27)
 				)
-				(hide yes)
 			)
 		)
-		(property "Value" "1N5819"
+		(property "Value" "BAT60B"
 			(at 68.8975 114.3 0)
 			(effects
@@
 			)
 		)
-		(property "Comment" ""
+		(property "Comment" "Alternative: 1N5819"
 			(at 68.58 118.11 0)
 			(effects
@@
 	)
 	(symbol
-		(lib_id "Regulator_Linear:AP2112K-3.3")
-		(at 95.25 120.65 0)
-		(unit 1)
-		(exclude_from_sim no)
-		(in_bom yes)
-		(on_board yes)
-		(dnp no)
-		(fields_autoplaced yes)
-		(property "Reference" "U4"
-			(at 95.25 111.76 0)
-			(effects
-				(font
-					(size 1.27 1.27)
-				)
-			)
-		)
-		(property "Value" "XC6220B331MR-G"
-			(at 95.25 114.3 0)
-			(effects
-				(font
-					(size 1.27 1.27)
-				)
-			)
-		)
-		(property "Footprint" "PCM_Package_TO_SOT_SMD_AKL:SOT-23-5"
-			(at 95.25 112.395 0)
-			(effects
-				(font
-					(size 1.27 1.27)
-				)
-				(hide yes)
-			)
-		)
-		(property "Datasheet" "https://product.torexsemi.com/system/files/series/xc6220.pdf"
-			(at 95.25 118.11 0)
-			(effects
-				(font
-					(size 1.27 1.27)
-				)
-				(hide yes)
-			)
-		)
-		(property "Description" ""
-			(at 95.25 120.65 0)
-			(effects
-				(font
-					(size 1.27 1.27)
-				)
-				(hide yes)
-			)
-		)
-		(property "Comment" ""
-			(at 95.25 120.65 0)
-			(effects
-				(font
-					(size 1.27 1.27)
-				)
-				(hide yes)
-			)
-		)
-		(pin "1"
-		)
-		(pin "2"
-		)
-		(pin "3"
-		)
-		(pin "4"
-		)
-		(pin "5"
-		)
-		(instances
-			(project "keyboard_right"
-				(path "/852dabbf-de45-4470-8176-59d37a754407"
-					(reference "U4")
-					(unit 1)
-				)
-			)
-			(project "nrfmicro"
-				(path "/bfc0aadc-38cf-466e-a642-68fdc3138c78"
-					(reference "U2")
-					(unit 1)
-				)
-			)
-		)
-	)
-	(symbol
 		(lib_id "power:VCC")
 		(at 86.36 182.88 180)
@@
 					(unit 1)
 				)
+			)
+		)
+	)
+	(symbol
+		(lib_id "Regulator_Linear:AP2112K-3.3")
+		(at 95.25 120.65 0)
+		(unit 1)
+		(exclude_from_sim no)
+		(in_bom yes)
+		(on_board yes)
+		(dnp no)
+		(fields_autoplaced yes)
+		(property "Reference" "U4"
+			(at 95.25 111.76 0)
+			(effects
+				(font
+					(size 1.27 1.27)
+				)
+			)
+		)
+		(property "Value" "XC6220B331MR-G"
+			(at 95.25 114.3 0)
+			(effects
+				(font
+					(size 1.27 1.27)
+				)
+			)
+		)
+		(property "Footprint" "PCM_Package_TO_SOT_SMD_AKL:SOT-23-5"
+			(at 95.25 112.395 0)
+			(effects
+				(font
+					(size 1.27 1.27)
+				)
+				(hide yes)
+			)
+		)
+		(property "Datasheet" "https://product.torexsemi.com/system/files/series/xc6220.pdf"
+			(at 95.25 118.11 0)
+			(effects
+				(font
+					(size 1.27 1.27)
+				)
+				(hide yes)
+			)
+		)
+		(property "Description" ""
+			(at 95.25 120.65 0)
+			(effects
+				(font
+					(size 1.27 1.27)
+				)
+				(hide yes)
+			)
+		)
+		(property "Comment" "Alternative: AP2112K"
+			(at 95.25 120.65 0)
+			(effects
+				(font
+					(size 1.27 1.27)
+				)
+				(hide yes)
+			)
+		)
+		(pin "1"
+		)
+		(pin "2"
+		)
+		(pin "3"
+		)
+		(pin "4"
+		)
+		(pin "5"
+		)
+		(instances
+			(project "keyboard_right"
+				(path "/852dabbf-de45-4470-8176-59d37a754407"
+					(reference "U4")
+					(unit 1)
+				)

Commit message: stencil temp
Parts:
- removed J4: HRS_FH34SRJ-06S-0.5SH(50), ec_parts:CONN6x1_FH34SRJ-6S-0.5SH50_HIR, symbol Connector_Generic_MountingPin:Conn_01x06_MountingPin
Connections:
- no-connect marks 10 -> 9
Other:
- note removed: "FFC Connector for Extra daughter board"
- note removed: "Pin functionalities. PA4 | |SPI1_NSS |SPI3_NSS | |USART2_CK PB3 | |SPI1_SCK |SPI3_SCK | |USART2_TX PB4 | |SPI1_MISO|SPI3_MISO| |USART2_RX PB5 | |SPI1_MOSI|SPI3_MOSI| |USART2_CK"
- moved on the sheet: FB1, R4, R5, R8

Commit message: Rev 2.1
Parts:
- added J4: HRS_FH34SRJ-06S-0.5SH(50), ec_parts:CONN6x1_FH12S-6S-1SH55, symbol Connector_Generic_MountingPin:Conn_01x06_MountingPin
Connections:
- net +3V3: now also J4.6 (Pin_6)
- net GND: now also J4.1 (Pin_1)
- net PA4: now also J4.5 (Pin_5)
- net PB3: now also J4.4 (Pin_4)
- net PB4: now also J4.3 (Pin_3)
- net PB5: now also J4.2 (Pin_2)
- no-connect marks 9 -> 10
Other:
- note added: "FFC Connector for Extra daughter board"
- note added: "Pin functionalities. PA4 | |SPI1_NSS |SPI3_NSS | |USART2_CK PB3 | |SPI1_SCK |SPI3_SCK | |USART2_TX PB4 | |SPI1_MISO|SPI3_MISO| |USART2_RX PB5 | |SPI1_MOSI|SPI3_MOSI| |USART2_CK"
- moved on the sheet: FB1, R4, R5, R8
