File: hardware/pcb/wheel/wheel.kicad_pcb (KiCad board)
At the start: 2 copper layers, 20.2 x 35.9 mm, 16 parts, among them J4 HRS_FH34SRJ-06S-0.5SH(50), SW1 RotaryEncoder_Switch, SW2 RotaryEncoder_Switch

Commit message: production
Changed lines of the file:
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@@
 	(net 5 "unconnected-(J4-MountPin-PadMP)")
 	(net 6 "GND")
-	(net 7 "unconnected-(J4-MountPin-PadMP)_1")
-	(net 8 "+3.3V")
-	(net 9 "Net-(R4-Pad2)")
-	(net 10 "Net-(R5-Pad2)")
-	(net 11 "Net-(R6-Pad1)")
-	(net 12 "Net-(R7-Pad2)")
-	(net 13 "Net-(R8-Pad2)")
-	(net 14 "Net-(R9-Pad1)")
+	(net 7 "+3.3V")
+	(net 8 "Net-(R4-Pad2)")
+	(net 9 "Net-(R5-Pad2)")
+	(net 10 "Net-(R6-Pad1)")
+	(net 11 "Net-(R7-Pad2)")
+	(net 12 "Net-(R8-Pad2)")
+	(net 13 "Net-(R9-Pad1)")
 	(footprint "ec_parts:CONN6x1_FH34SRJ-6S-0.5SH50_HIR"
 		(locked yes)
@@
 			(size 0.3556 0.8382)
 			(layers "F.Cu" "F.Mask" "F.Paste")
-			(net 8 "+3.3V")
+			(net 7 "+3.3V")
 			(pinfunction "Pin_6")
 			(pintype "passive")
@@
 			(size 0.4064 0.8382)
 			(layers "F.Cu" "F.Mask" "F.Paste")
-			(net 7 "unconnected-(J4-MountPin-PadMP)_1")
+			(net 5 "unconnected-(J4-MountPin-PadMP)")
 			(pinfunction "MountPin")
 			(pintype "passive+no_connect")
@@
 			(layers "F.Cu" "F.Mask" "F.Paste")
 			(roundrect_rratio 0.25)
-			(net 12 "Net-(R7-Pad2)")
+			(net 11 "Net-(R7-Pad2)")
 			(pintype "passive")
 		)
@@
 		(sheetfile "wheel.kicad_sch")
 		(attr exclude_from_pos_files)
-		(pad "1" thru_hole circle
+		(pad "" np_thru_hole circle
 			(at 0 0)
-			(size 4.2 4.2)
-			(drill 2.5)
+			(size 1.62 1.62)
+			(drill 1.62)
 			(layers "*.Cu" "*.Mask")
-			(remove_unused_layers no)
 		)
 		(embedded_fonts no)
@@
 			(layers "F.Cu" "F.Mask" "F.Paste")
 			(roundrect_rratio 0.25)
-			(net 13 "Net-(R8-Pad2)")
+			(net 12 "Net-(R8-Pad2)")
 			(pintype "passive")
 		)
@@
 			(layers "F.Cu" "F.Mask" "F.Paste")
 			(roundrect_rratio 0.25)
-			(net 9 "Net-(R4-Pad2)")
+			(net 8 "Net-(R4-Pad2)")
 			(pintype "passive")
 		)
@@
 			(layers "F.Cu" "F.Mask" "F.Paste")
 			(roundrect_rratio 0.25)
-			(net 11 "Net-(R6-Pad1)")
+			(net 10 "Net-(R6-Pad1)")
 			(pintype "passive")
 		)
@@
 		(sheetfile "wheel.kicad_sch")
 		(attr exclude_from_pos_files)
-		(pad "1" thru_hole circle
+		(pad "" np_thru_hole circle
 			(at 0 0)
-			(size 4.2 4.2)
-			(drill 2.5)
+			(size 1.62 1.62)
+			(drill 1.62)
 			(layers "*.Cu" "*.Mask")
-			(remove_unused_layers no)
 		)
 		(embedded_fonts no)
@@
 			(layers "F.Cu" "F.Mask" "F.Paste")
 			(roundrect_rratio 0.25)
-			(net 8 "+3.3V")
+			(net 7 "+3.3V")
 			(pintype "passive")
 		)
@@
 			(layers "F.Cu" "F.Mask" "F.Paste")
 			(roundrect_rratio 0.25)
-			(net 10 "Net-(R5-Pad2)")
+			(net 9 "Net-(R5-Pad2)")
 			(pintype "passive")
 		)
@@
 			(layers "*.Cu" "*.Mask")
 			(remove_unused_layers no)
-			(net 9 "Net-(R4-Pad2)")
+			(net 8 "Net-(R4-Pad2)")
 			(pinfunction "A")
 			(pintype "passive")
@@
 			(layers "*.Cu" "*.Mask")
 			(remove_unused_layers no)
-			(net 10 "Net-(R5-Pad2)")
+			(net 9 "Net-(R5-Pad2)")
 			(pinfunction "B")
 			(pintype "passive")
@@
 			(layers "*.Cu" "*.Mask")
 			(remove_unused_layers no)
-			(net 11 "Net-(R6-Pad1)")
+			(net 10 "Net-(R6-Pad1)")
 			(pinfunction "S2")
 			(pintype "passive")
@@
 		(sheetfile "wheel.kicad_sch")
 		(attr exclude_from_pos_files)
-		(pad "1" thru_hole circle
+		(pad "" np_thru_hole circle
 			(at 0 0)
-			(size 4.2 4.2)
-			(drill 2.5)
+			(size 1.62 1.62)
+			(drill 1.62)
 			(layers "*.Cu" "*.Mask")
-			(remove_unused_layers no)
 		)
 		(embedded_fonts no)
@@
 			(layers "F.Cu" "F.Mask" "F.Paste")
 			(roundrect_rratio 0.25)
-			(net 8 "+3.3V")
+			(net 7 "+3.3V")
 			(pintype "passive")
 		)
@@
 			(layers "F.Cu" "F.Mask" "F.Paste")
 			(roundrect_rratio 0.25)
-			(net 8 "+3.3V")
+			(net 7 "+3.3V")
 			(pintype "passive")
 		)
@@
 		(sheetfile "wheel.kicad_sch")
 		(attr exclude_from_pos_files)
-		(pad "1" thru_hole circle
+		(pad "" np_thru_hole circle
 			(at 0 0)
-			(size 4.2 4.2)
-			(drill 2.5)
+			(size 1.62 1.62)
+			(drill 1.62)
 			(layers "*.Cu" "*.Mask")
-			(remove_unused_layers no)
 		)
 		(embedded_fonts no)
@@
 			(layers "F.Cu" "F.Mask" "F.Paste")
 			(roundrect_rratio 0.25)
-			(net 14 "Net-(R9-Pad1)")
+			(net 13 "Net-(R9-Pad1)")
 			(pintype "passive")
 		)
@@
 			(layers "*.Cu" "*.Mask")
 			(remove_unused_layers no)
-			(net 12 "Net-(R7-Pad2)")
+			(net 11 "Net-(R7-Pad2)")
 			(pinfunction "A")
 			(pintype "passive")
@@
 			(layers "*.Cu" "*.Mask")
 			(remove_unused_layers no)
-			(net 13 "Net-(R8-Pad2)")
+			(net 12 "Net-(R8-Pad2)")
 			(pinfunction "B")
 			(pintype "passive")
@@
 			(layers "*.Cu" "*.Mask")
 			(remove_unused_layers no)
-			(net 14 "Net-(R9-Pad1)")
+			(net 13 "Net-(R9-Pad1)")
 			(pinfunction "S2")
 			(pintype "passive")
@@
 		(width 0.5)
 		(layer "F.Cu")
-		(net 8)
+		(net 7)
 	)
 	(segment
@@
 		(width 0.5)
 		(layer "F.Cu")
-		(net 8)
+		(net 7)
 	)
 	(segment
@@
 		(width 0.5)
 		(layer "F.Cu")
-		(net 8)
+		(net 7)
 	)
 	(segment
@@
 		(width 0.5)
 		(layer "F.Cu")
-		(net 8)
+		(net 7)
 	)
 	(arc
@@
 		(width 0.5)
 		(layer "F.Cu")
-		(net 8)
+		(net 7)
 	)
 	(segment
@@
 		(width 0.3)
 		(layer "F.Cu")
-		(net 9)
+		(net 8)
 	)
 	(segment
@@
 		(width 0.3)
 		(layer "F.Cu")
-		(net 9)
+		(net 8)
 	)
 	(arc
@@
 		(width 0.3)
 		(layer "F.Cu")
-		(net 9)
+		(net 8)
 	)
 	(via
@@
 		(drill 0.3)
 		(layers "F.Cu" "B.Cu")
-		(net 10)
+		(net 9)
 	)
 	(segment
@@
 		(width 0.3)
 		(layer "B.Cu")
-		(net 10)
+		(net 9)
 	)
 	(segment
@@
 		(width 0.3)
 		(layer "B.Cu")
-		(net 10)
+		(net 9)
 	)
 	(segment
@@
 		(width 0.3)
 		(layer "B.Cu")
-		(net 10)
+		(net 9)
 	)
 	(arc
@@
 		(width 0.3)
 		(layer "B.Cu")
-		(net 10)
+		(net 9)
 	)
 	(arc
@@
 		(width 0.3)
 		(layer "B.Cu")
-		(net 10)
+		(net 9)
 	)
 	(segment
@@
 		(width 0.3)
 		(layer "F.Cu")
-		(net 11)
+		(net 10)
 	)
 	(segment
@@
 		(width 0.3)
 		(layer "F.Cu")
-		(net 11)
+		(net 10)
 	)
 	(arc
@@
 		(width 0.3)
 		(layer "F.Cu")
-		(net 11)
+		(net 10)
 	)
 	(arc
@@
 		(width 0.3)
 		(layer "F.Cu")
-		(net 11)
+		(net 10)
 	)
 	(segment
@@
 		(width 0.3)
 		(layer "F.Cu")
-		(net 12)
+		(net 11)
 	)
 	(segment
@@
 		(width 0.3)
 		(layer "F.Cu")
-		(net 12)
+		(net 11)
 	)
 	(arc
@@
 		(width 0.3)
 		(layer "F.Cu")
-		(net 12)
+		(net 11)
 	)
 	(via
@@
 		(drill 0.3)
 		(layers "F.Cu" "B.Cu")
-		(net 13)
+		(net 12)
 	)
 	(segment
@@
 		(width 0.3)
 		(layer "B.Cu")
-		(net 13)
+		(net 12)
 	)
 	(segment
@@
 		(width 0.3)
 		(layer "B.Cu")
-		(net 13)
+		(net 12)
 	)
 	(segment
@@
 		(width 0.3)
 		(layer "B.Cu")
-		(net 13)
+		(net 12)
 	)
 	(arc
@@
 		(width 0.3)
 		(layer "B.Cu")
-		(net 13)
+		(net 12)
 	)
 	(arc
@@
 		(width 0.3)
 		(layer "B.Cu")
-		(net 13)
+		(net 12)
 	)
 	(segment
@@
 		(width 0.3)
 		(layer "F.Cu")
-		(net 14)
+		(net 13)
 	)
 	(segment
@@
 		(width 0.3)
 		(layer "F.Cu")
-		(net 14)
+		(net 13)
 	)
 	(segment
@@
 		(width 0.3)
 		(layer "F.Cu")
-		(net 14)
+		(net 13)
 	)
 	(arc
@@
 		(width 0.3)
 		(layer "F.Cu")
-		(net 14)
+		(net 13)
 	)
 	(arc
@@
 		(width 0.3)
 		(layer "F.Cu")
-		(net 14)
+		(net 13)
 	)
 	(zone
