File: hardware/pcb/wheel/wheel.kicad_sch (KiCad schematic)
At the start: 16 parts, among them J4 HRS_FH34SRJ-06S-0.5SH(50), SW1 RotaryEncoder_Switch, SW2 RotaryEncoder_Switch

Commit message: production
Parts:
- H3, H4, H5, H6: footprint ec_parts:SMT-SO-M1.6-with-ring -> ec_parts:SMT-SO-M1.6-screwhole_only
Changed lines of the file:
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@@
 			)
 		)
-		(property "Footprint" "ec_parts:SMT-SO-M1.6-with-ring"
+		(property "Footprint" "ec_parts:SMT-SO-M1.6-screwhole_only"
 			(at 36.83 58.42 0)
 			(effects
@@
 			)
 		)
-		(property "Footprint" "ec_parts:SMT-SO-M1.6-with-ring"
+		(property "Footprint" "ec_parts:SMT-SO-M1.6-screwhole_only"
 			(at 53.34 58.42 0)
 			(effects
@@
 			)
 		)
-		(property "Footprint" "ec_parts:SMT-SO-M1.6-with-ring"
+		(property "Footprint" "ec_parts:SMT-SO-M1.6-screwhole_only"
 			(at 44.45 58.42 0)
 			(effects
@@
 			)
 		)
-		(property "Footprint" "ec_parts:SMT-SO-M1.6-with-ring"
+		(property "Footprint" "ec_parts:SMT-SO-M1.6-screwhole_only"
 			(at 60.96 58.42 0)
 			(effects
