File: hardware/pcb/wheel/wheel_panel.kicad_pcb (KiCad board)
At the start: 2 copper layers, 64.6 x 51.9 mm, 108 parts, among them J4 HRS_FH34SRJ-06S-0.5SH(50), SW1 RotaryEncoder_Switch, SW2 RotaryEncoder_Switch

Commit message: production
Parts:
- removed the R1 at (127.7, 35.6)
- removed the R1 at (172.1, 35.6)
- removed the R1 at (149.8, 35.6)
- removed the R2 at (126.2, 35.6)
- removed the R2 at (170.6, 35.6)
- removed the R2 at (148.3, 35.6)
- removed the R3 at (169.1, 35.6)
- removed the R3 at (124.7, 35.6)
- removed the R3 at (146.8, 35.6)
- removed the R4 at (167.7, 40.8)
- removed the R4 at (123.3, 40.8)
- removed the R4 at (145.5, 40.8)
- removed the R5 at (145.5, 39.3)
- removed the R5 at (167.7, 39.3)
- removed the R5 at (123.3, 39.3)
- removed the R6 at (145.5, 37.8)
- removed the R6 at (123.3, 37.8)
- removed the R6 at (167.7, 37.8)
- removed the R7 at (151.5, 40.8)
- removed the R7 at (173.7, 40.8)
- removed the R7 at (129.3, 40.8)
- removed the R8 at (173.7, 39.3)
- removed the R8 at (151.5, 39.3)
- removed the R8 at (129.3, 39.3)
- removed the R9 at (129.3, 37.8)
- removed the R9 at (151.5, 37.8)
- removed the R9 at (173.7, 37.8)
- added R1: 10k, PCM_Resistor_SMD_AKL:R_0603_1608Metric_Pad1.05x0.95mm_HandSolder, F.Cu at (172.1, 35.6)
- added R1: 10k, PCM_Resistor_SMD_AKL:R_0603_1608Metric_Pad1.05x0.95mm_HandSolder, F.Cu at (127.7, 35.6)
- added R1: 10k, PCM_Resistor_SMD_AKL:R_0603_1608Metric_Pad1.05x0.95mm_HandSolder, F.Cu at (149.8, 35.6)
- added R2: 10k, PCM_Resistor_SMD_AKL:R_0603_1608Metric_Pad1.05x0.95mm_HandSolder, F.Cu at (148.3, 35.6)
- added R2: 10k, PCM_Resistor_SMD_AKL:R_0603_1608Metric_Pad1.05x0.95mm_HandSolder, F.Cu at (170.6, 35.6)
- added R2: 10k, PCM_Resistor_SMD_AKL:R_0603_1608Metric_Pad1.05x0.95mm_HandSolder, F.Cu at (126.2, 35.6)
- added R3: 10k, PCM_Resistor_SMD_AKL:R_0603_1608Metric_Pad1.05x0.95mm_HandSolder, F.Cu at (124.7, 35.6)
- added R3: 10k, PCM_Resistor_SMD_AKL:R_0603_1608Metric_Pad1.05x0.95mm_HandSolder, F.Cu at (169.1, 35.6)
- added R3: 10k, PCM_Resistor_SMD_AKL:R_0603_1608Metric_Pad1.05x0.95mm_HandSolder, F.Cu at (146.8, 35.6)
- added R4: 0, PCM_Resistor_SMD_AKL:R_0603_1608Metric_Pad1.05x0.95mm_HandSolder, F.Cu at (167.7, 40.8)
- added R4: 0, PCM_Resistor_SMD_AKL:R_0603_1608Metric_Pad1.05x0.95mm_HandSolder, F.Cu at (123.3, 40.8)
- added R4: 0, PCM_Resistor_SMD_AKL:R_0603_1608Metric_Pad1.05x0.95mm_HandSolder, F.Cu at (145.5, 40.8)
- added R5: 0, PCM_Resistor_SMD_AKL:R_0603_1608Metric_Pad1.05x0.95mm_HandSolder, F.Cu at (167.7, 39.3)
- added R5: 0, PCM_Resistor_SMD_AKL:R_0603_1608Metric_Pad1.05x0.95mm_HandSolder, F.Cu at (123.3, 39.3)
- added R5: 0, PCM_Resistor_SMD_AKL:R_0603_1608Metric_Pad1.05x0.95mm_HandSolder, F.Cu at (145.5, 39.3)
- added R6: 0, PCM_Resistor_SMD_AKL:R_0603_1608Metric_Pad1.05x0.95mm_HandSolder, F.Cu at (145.5, 37.8)
- added R6: 0, PCM_Resistor_SMD_AKL:R_0603_1608Metric_Pad1.05x0.95mm_HandSolder, F.Cu at (167.7, 37.8)
- added R6: 0, PCM_Resistor_SMD_AKL:R_0603_1608Metric_Pad1.05x0.95mm_HandSolder, F.Cu at (123.3, 37.8)
- added R7: 0, PCM_Resistor_SMD_AKL:R_0603_1608Metric_Pad1.05x0.95mm_HandSolder, F.Cu at (173.7, 40.8)
- added R7: 0, PCM_Resistor_SMD_AKL:R_0603_1608Metric_Pad1.05x0.95mm_HandSolder, F.Cu at (151.5, 40.8)
- added R7: 0, PCM_Resistor_SMD_AKL:R_0603_1608Metric_Pad1.05x0.95mm_HandSolder, F.Cu at (129.3, 40.8)
- added R8: 0, PCM_Resistor_SMD_AKL:R_0603_1608Metric_Pad1.05x0.95mm_HandSolder, F.Cu at (173.7, 39.3)
- added R8: 0, PCM_Resistor_SMD_AKL:R_0603_1608Metric_Pad1.05x0.95mm_HandSolder, F.Cu at (151.5, 39.3)
- added R8: 0, PCM_Resistor_SMD_AKL:R_0603_1608Metric_Pad1.05x0.95mm_HandSolder, F.Cu at (129.3, 39.3)
- added R9: 0, PCM_Resistor_SMD_AKL:R_0603_1608Metric_Pad1.05x0.95mm_HandSolder, F.Cu at (151.5, 37.8)
- added R9: 0, PCM_Resistor_SMD_AKL:R_0603_1608Metric_Pad1.05x0.95mm_HandSolder, F.Cu at (173.7, 37.8)
- added R9: 0, PCM_Resistor_SMD_AKL:R_0603_1608Metric_Pad1.05x0.95mm_HandSolder, F.Cu at (129.3, 37.8)
Connections:
- net Board_0-unconnected-(J4-MountPin-PadMP)_1 renamed Board_0-unconnected-(J4-MountPin-PadMP)
- net Board_1-unconnected-(J4-MountPin-PadMP)_1 renamed Board_1-unconnected-(J4-MountPin-PadMP)
- net Board_2-unconnected-(J4-MountPin-PadMP)_1 renamed Board_2-unconnected-(J4-MountPin-PadMP)
Routing:
- net Board_2-ACCS_2: track 15.3 -> 14.5 mm
- net Board_1-ACCS_2: track 15.3 -> 14.5 mm
- net Board_0-ACCS_2: track 15.3 -> 14.5 mm
