File: hardware/case/kicad/case.kicad_pcb (KiCad board)
At the start: 2 copper layers, 133.8 x 110.4 mm, 52 parts, among them J1 SM03B-SRSS-TB, J2 PJ320D, J3 HRO_TYPE-C-31-M-12, SW29 PTS845

Commit message: Rev 2.1
Other:
- board size 133.8 x 110.4 mm -> 143.8 x 121.9 mm
